File: DAWG_ServoDriver.kicad_sch (KiCad schematic)
At the start: 89 parts, among them J1 Conn_01x04_Pin, J2 Conn_01x12_seperated, J3 Conn_01x12_seperated, J4 Conn_01x12_seperated, J5 Conn_01x12_seperated, J6 Conn_01x12_seperated, Q1 BSS138, Q10 BSS138, Q11 BSS138, Q12 BSS138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

Commit message: feedback
Other:
- note added: "- No connector for battery (2 screw-terminal for battery) - no pins for nucleo-64 board - no need for another LIDAR I2C pull up lines (one already provided)"
- note added: "Good recommendation in STM32 datasheets is to put a 0.1uF per VDD pin (total 5 pins taking 3.3V, 4 0.1uF placed). 4.7uF could be also replaced by 10uF (we have them already)"
- note added: "Isn't it better to connect NOT SLEEP to GND ?"
- note added: "Lidar takes 5V in, however what voltage is on the I2C ? we probably need to have here a logic level converter (3.3/5V) ?"
- note added: "NRST is pulled up internally, however we would like to have some button that would reset it. the low-pass is there (0.1uF and internal pull-up), just need to add a button to ground (or button + another resistor)"
- note added: "PWM17/1 seems unconnected also not sure whether we want to use TIM 17"
- note added: "PWM4/3 is not placed. There does not seem to be any pin conflict and TIM4/3 can be placed ?"
- note added: "Strong assumption that the power from screw-terminal will power the servos. Is that what we agreed on ?"
- note added: "This line will power STM32 no? should be connected to 3.3V"
- note added: "could be pulled to GND (set LSB to 0)"
- note added: "no value selected. could be > 1uF"
- note added: "probably should be routed : we should use interrupt based comms (no polling ).FSYNC should be connected to GND."
- note added: "uncommon value of resistors. Could be 1.8k, 2.2k or 4.7"
