File: DAWG_ServoDriver.kicad_sch (KiCad schematic)
At the start: 89 parts, among them J1 Conn_01x04_Pin, J2 Conn_01x12_seperated, J3 Conn_01x12_seperated, J4 Conn_01x12_seperated, J5 Conn_01x12_seperated, J6 Conn_01x12_seperated, Q1 BSS138, Q10 BSS138, Q11 BSS138, Q12 BSS138, Q13 BSS138, Q14 BSS138, Q15 BSS138, Q16 BSS138, Q17 BSS138, Q18 BSS138, Q2 BSS138, Q3 BSS138, Q4 BSS138, Q5 BSS138, Q6 BSS138, Q7 BSS138, Q8 BSS138, Q9 BSS138, SW1 SW_SPDT, U1 STM32G431C8Tx, U3 TPS62177DQC, U4 ICM-20602, U6 LD1117S12TR_SOT223, Y1 Crystal_GND24

Commit message: Your commit message
Parts:
- added R3, R4: 2k2, symbol Device:R
- added SW2: SW_Push, symbol Switch:SW_Push
- C18: value C -> 100n
- C5: value 4.7u -> 10u
- R54, R55: value 3k -> 2k2
Connections:
- net PWM17/1 is gone; now on net PWM1/1: U1.15 (PA7)
- net +3.3V: now also R3.1, R4.1
- net GND: now also U3.8 (~{SLEEP}), U4.8 (FSYNC), SW2.2
- net I2C1_SCL: no longer LiDAR-V1.4 (SCL)
- net I2C1_SDA: no longer LiDAR-V1.3 (SDA)
- net NRST: now also SW2.1
- net PWM1/1: no longer U1.30 (PA8)
- net I2C3_SDA: now reaches U1.42 (PB5)
- net I2C3_SDA: now also LiDAR-V1.3 (SDA), R3.2
- net 3Vout renamed 3.3Vout
- net 3.3Vout: no longer U3.8 (~{SLEEP})
- new net I2C3_SCL: LiDAR-V1.4 (SCL), R4.2, U1.30 (PA8)
- no-connect marks 15 -> 14
Other:
- moved on the sheet: C1, C12, C13, C18, C2, C20, C3, C4, C5, C9, J1, J2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

Commit message: Updated IMU, Added Motor Drivers and screw terminal, Added the morpho header
Parts:
- added C21: 10n, symbol Device:C
- added C22, C25, C27, C29, C31, C7: 0.1u, symbol Device:C
- added C23, C24: 680u, symbol Device:C_Polarized_Small_US
- added C26, C28, C30, C32: 47u, symbol Device:C
- added C6: 100n, symbol Device:C
- added C8: 2.2u, symbol Device:C
- added CN1, CN2: Conn_02x19_Odd_Even, Connector_PinSocket_2.54mm:PinSocket_2x19_P2.54mm_Vertical, symbol Connector_Generic:Conn_02x19_Odd_Even
- added IC1, IC2, IC3, IC4: DRV8251ADDAR, SOIC127P600X170-9N, symbol Driver_Motor:DRV8251ADDAR
- added J10, J11, J12, J9: Screw_Terminal_01x02, symbol Connector:Screw_Terminal_01x02
- added J7, J8: Screw_Terminal_01x02, TerminalBlock_MetzConnect:TerminalBlock_MetzConnect_Type701_RT11L02HGLU_1x02_P6.35mm_Horizontal, symbol Connector:Screw_Terminal_01x02
- added Q19, Q20: BSS138, Package_TO_SOT_SMD:SOT-23, symbol Transistor_FET:BSS138
- added R10, R9: R, symbol Device:R
- added R5, R6, R7, R8: 10k, symbol Device:R
- added U2: ICM-20602, Package_LGA:LGA-16_3x3mm_P0.5mm_LayoutBorder3x5y, symbol Sensor_Motion:ICM-20602
- R3, R4: value 2k2 -> R
Connections:
- net 3.3Vout is gone; now on net +3.3V: C11.1, L1.2, Q1.1 (G), Q10.1 (G), Q11.1 (G), Q12.1 (G), Q13.1 (G), Q14.1 (G), Q15.1 (G), Q16.1 (G), Q17.1 (G), Q18.1 (G), Q2.1 (G), Q3.1 (G), Q4.1 (G), Q5.1 (G), Q6.1 (G), Q7.1 (G), Q8.1 (G), Q9.1 (G), R18.2, R2.1, R21.2, R23.2, R25.2, R27.2, R29.2, R31.2, R33.2, R35.2, R37.2, R39.2, R41.2, R43.2, R45.2, R47.2, R49.2, R51.2, R53.2, U3.10 (VOS)
- net +3.3V: now also C21.1, C6.1, C7.1, C8.1, CN1.16 (Pin_16), IC1.4 (VREF), IC2.4 (VREF), IC3.4 (VREF), IC4.4 (VREF), R5.2, R7.2, U2.1 (VDDIO), U2.16 (VDD), U2.4 (SAO/SD0), U2.5 (~{CS}); no longer R3.1, R4.1, U4.4 (SAO/SD0)
- net GND: now also U4.4 (SAO/SD0), C21.2, C22.1, C23.2, C24.2, C25.1, C26.1, C27.1, C28.1, C29.1, C30.1, C31.1, C32.1, C6.2, C7.2, C8.2, CN1.20 (Pin_20), CN1.22 (Pin_22), IC1.7 (GND_1), IC1.9 (GND_2), IC2.7 (GND_1), IC2.9 (GND_2), IC3.7 (GND_1), IC3.9 (GND_2), IC4.7 (GND_1), IC4.9 (GND_2), J7.2 (Pin_2), J8.2 (Pin_2), U2.10 (GND), U2.11 (GND), U2.12 (GND), U2.13 (GND), U2.15 (GND), U2.8 (FSYNC), U2.9 (GND)
- net I2C1_SCL: now also CN2.3 (Pin_3), Q20.2 (S), R8.1, U2.2 (SCL/SPC)
- net I2C1_SDA: now also CN2.5 (Pin_5), Q19.2 (S), Q19.3 (D), R5.1, R6.1, U2.3 (SDA/SDI)
- net I2C3_SCL: no longer R4.2
- net I2C3_SDA: no longer R3.2
- net PWM1/1: now also CN2.23 (Pin_23)
- net PWM1/2: now also CN2.21 (Pin_21)
- net PWM2/1: now also CN2.11 (Pin_11), IC1.2 (IN2), IC2.2 (IN2), IC3.2 (IN2), IC4.2 (IN2)
- net PWM2/3: now also CN2.25 (Pin_25)
- net PWM3/1: now also CN2.13 (Pin_13), IC1.3 (IN1), IC2.3 (IN1), IC3.3 (IN1), IC4.3 (IN1)
- net PWM3/2: now also CN2.19 (Pin_19), CN2.29 (Pin_29)
- net PWM4/1: now also CN2.17 (Pin_17)
- net IMU1_INT: now reaches U4.6 (INT)
- net IMU1_INT: now also CN2.12 (Pin_12)
- net 5Vout renamed +5V
- net +5V: now also C25.2, C26.2, C27.2, C28.2, C29.2, C30.2, C31.2, C32.2, CN1.18 (Pin_18), IC1.5 (VM), IC2.5 (VM), IC3.5 (VM), IC4.5 (VM), Q19.1 (G), Q20.1 (G), R6.2, R8.2
- net Vbatt renamed +BATT
- new net: C22.2, U2.14 (REGOUT)
- new net: IC3.1 (IPROPI), R9.2
- new net: IC4.1 (IPROPI), R10.2
- new net: IC1.1 (IPROPI), R3.2
- new net: IC2.1 (IPROPI), R4.2
- new net ADC1/14: CN2.34 (Pin_34), R3.1
- new net ADC1/15: CN2.6 (Pin_6), R4.1
- new net ADC1/7: CN2.15 (Pin_15), R10.1
- new net ADC1/9: CN2.24 (Pin_24), R9.1
- new net IMU2_INT: CN2.16 (Pin_16), U2.6 (INT)
- new net V_DCMotor: C24.1, J8.1 (Pin_1)
- new net V_LIDAR2: Q20.3 (D), R7.1
- new net V_M1A: IC1.8 (OUT2), J9.1 (Pin_1)
- new net V_M1B: IC1.6 (OUT1), J9.2 (Pin_2)
- new net V_M2A: IC2.8 (OUT2), J10.1 (Pin_1)
- new net V_M2B: IC2.6 (OUT1), J10.2 (Pin_2)
- new net V_M3A: IC3.8 (OUT2), J11.1 (Pin_1)
- new net V_M3B: IC3.6 (OUT1), J11.2 (Pin_2)
- new net V_M4A: IC4.8 (OUT2), J12.1 (Pin_1)
- new net V_M4B: IC4.6 (OUT1), J12.2 (Pin_2)
- new net V_Servo: C23.1, J7.1 (Pin_1)
- no-connect marks 14 -> 12
Other:
- note added: "IMU1"
- note added: "IMU2"
- note added: "Morpho Header"
- note added: "Motor Driver"
- note removed: "IMU"
- note removed: "Notes Missing: - C18 how to determine? - Instead of the bead what should be added? - The LiDAR I2C and SDA are not connected to pull up resistors"
- moved on the sheet: C1, C10, C11, C12, C13, C14, C15, C16, C17, C18, C19, C2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

Commit message: Added motor driver resistor values and arranged components
Parts:
- R10, R3, R4, R9: value R -> 1k5
Other:
- note added: "Logic Level Converters"
- note added: "Motor Terminals"
- note added: "Power"
- note added: "Power Terminals"
- note removed: "Logic Level Converter"
- note removed: "Power Conversion"
- moved on the sheet: C1, C10, C11, C12, C13, C14, C15, C16, C17, C18, C19, C2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

Commit message: Added footprints for all except SW1, SW2, ServoHeader, crystal
Parts:
- removed J12: Screw_Terminal_01x02, symbol Connector:Screw_Terminal_01x02
- removed R10, R3, R4, R9: 1k5, symbol Device:R
- removed R5, R6, R7, R8: 10k, symbol Device:R
- added J12: Conn_01x03, Connector_PinHeader_1.00mm:PinHeader_1x03_P1.00mm_Vertical_SMD_Pin1Left, symbol Connector_Generic:Conn_01x03
- added J4, J5, J6, J7: Conn_01x05, TerminalBlock_MetzConnect:TerminalBlock_MetzConnect_Type011_RT05505HBWC_1x05_P5.00mm_Horizontal, symbol Connector:Screw_Terminal_01x05
- added J8: Screw_Terminal_01x02, TerminalBlock_MetzConnect:TerminalBlock_MetzConnect_Type011_RT05502HBWC_1x02_P5.00mm_Horizontal, symbol Connector:Screw_Terminal_01x02
- added R41, R42, R43, R44: 1k5, Resistor_SMD:R_0402_1005Metric_Pad0.72x0.64mm_HandSolder, symbol Device:R
- added R45, R46, R47, R48: 10k, Resistor_SMD:R_0402_1005Metric_Pad0.72x0.64mm_HandSolder, symbol Device:R
- C1: renamed from C5; footprint (none) -> Capacitor_SMD:C_0402_1005Metric_Pad0.74x0.62mm_HandSolder
- C10, C4: footprint (none) -> Capacitor_SMD:C_0402_1005Metric_Pad0.74x0.62mm_HandSolder
- C11: renamed from C18; footprint (none) -> Capacitor_SMD:C_0402_1005Metric_Pad0.74x0.62mm_HandSolder
- C12: renamed from C15; value 0.1u -> 100n; footprint (none) -> Capacitor_SMD:C_0402_1005Metric_Pad0.74x0.62mm_HandSolder
- C13: renamed from C7; value 0.1u -> 100n; footprint (none) -> Capacitor_SMD:C_0402_1005Metric_Pad0.74x0.62mm_HandSolder
- C14: renamed from C24; footprint (none) -> Capacitor_SMD:CP_Elec_10x10.5
- C15: renamed from C14; footprint (none) -> Capacitor_SMD:C_0402_1005Metric_Pad0.74x0.62mm_HandSolder
- C16: renamed from C8; footprint (none) -> Capacitor_SMD:C_0402_1005Metric_Pad0.74x0.62mm_HandSolder
- C17: renamed from C23; footprint (none) -> Capacitor_SMD:CP_Elec_10x10.5
- C18: renamed from C19; footprint (none) -> Capacitor_SMD:C_0402_1005Metric_Pad0.74x0.62mm_HandSolder
- C19: renamed from C17; footprint (none) -> Capacitor_SMD:C_0402_1005Metric_Pad0.74x0.62mm_HandSolder
- C2: renamed from C6; footprint (none) -> Capacitor_SMD:C_0402_1005Metric_Pad0.74x0.62mm_HandSolder
- C20: renamed from C21; footprint (none) -> Capacitor_SMD:C_0402_1005Metric_Pad0.74x0.62mm_HandSolder
- C21: renamed from C16; value 0.1u -> 100n; footprint (none) -> Capacitor_SMD:C_0402_1005Metric_Pad0.74x0.62mm_HandSolder
- C22, C25, C27: value 0.1u -> 100n; footprint (none) -> Capacitor_SMD:C_0402_1005Metric_Pad0.74x0.62mm_HandSolder
- C23: renamed from C11; footprint (none) -> Capacitor_SMD:C_0402_1005Metric_Pad0.74x0.62mm_HandSolder
- C24: renamed from C20; footprint (none) -> Capacitor_SMD:CP_Elec_10x10.5
- C26, C28: value 47u -> 100n; footprint (none) -> Capacitor_SMD:C_0402_1005Metric_Pad0.74x0.62mm_HandSolder
- C29, C31: value 0.1u -> 47u; footprint (none) -> Capacitor_SMD:C_1206_3216Metric_Pad1.33x1.80mm_HandSolder
- C3: renamed from C9; footprint (none) -> Capacitor_SMD:C_0402_1005Metric_Pad0.74x0.62mm_HandSolder
- C30, C32: footprint (none) -> Capacitor_SMD:C_1206_3216Metric_Pad1.33x1.80mm_HandSolder
- C5: renamed from C12; footprint (none) -> Capacitor_SMD:C_0402_1005Metric_Pad0.74x0.62mm_HandSolder
- C6: renamed from C3; footprint (none) -> Capacitor_SMD:C_0402_1005Metric_Pad0.74x0.62mm_HandSolder
- C7: renamed from C13; footprint (none) -> Capacitor_SMD:C_0402_1005Metric_Pad0.74x0.62mm_HandSolder
- C8: renamed from C2; footprint (none) -> Capacitor_SMD:C_0402_1005Metric_Pad0.74x0.62mm_HandSolder
- C9: renamed from C1; footprint (none) -> Capacitor_SMD:C_0402_1005Metric_Pad0.74x0.62mm_HandSolder
- IC1, IC2, IC3, IC4: footprint SOIC127P600X170-9N -> DAWG_PCBFootprints:SOIC127P600X170-9N
- J1: footprint (none) -> Connector_PinHeader_1.00mm:PinHeader_1x04_P1.00mm_Vertical_SMD_Pin1Left
- J10, J11, J9: footprint (none) -> TerminalBlock_MetzConnect:TerminalBlock_MetzConnect_Type011_RT05502HBWC_1x02_P5.00mm_Horizontal
- J13: renamed from J2; footprint (none) -> Connector_PinHeader_1.00mm:PinHeader_1x12_P1.00mm_Vertical_SMD_Pin1Right
- J14: renamed from J4; footprint (none) -> Connector_PinHeader_1.00mm:PinHeader_1x12_P1.00mm_Vertical_SMD_Pin1Right
- J15: renamed from J6; footprint (none) -> Connector_PinHeader_1.00mm:PinHeader_1x06_P1.00mm_Vertical_SMD_Pin1Left
- J17: renamed from J5; footprint (none) -> Connector_PinHeader_1.00mm:PinHeader_1x12_P1.00mm_Vertical_SMD_Pin1Right
- L1: footprint (none) -> Inductor_SMD:L_0402_1005Metric_Pad0.77x0.64mm_HandSolder
- R1: renamed from R19; footprint (none) -> Resistor_SMD:R_0402_1005Metric_Pad0.72x0.64mm_HandSolder
- R10: renamed from R40; footprint (none) -> Resistor_SMD:R_0402_1005Metric_Pad0.72x0.64mm_HandSolder
- R11: renamed from R23; footprint (none) -> Resistor_SMD:R_0402_1005Metric_Pad0.72x0.64mm_HandSolder
- R12: renamed from R41; footprint (none) -> Resistor_SMD:R_0402_1005Metric_Pad0.72x0.64mm_HandSolder
- R13: renamed from R1; footprint (none) -> Resistor_SMD:R_0402_1005Metric_Pad0.72x0.64mm_HandSolder
- R14: renamed from R24; footprint (none) -> Resistor_SMD:R_0402_1005Metric_Pad0.72x0.64mm_HandSolder
- R15: renamed from R42; footprint (none) -> Resistor_SMD:R_0402_1005Metric_Pad0.72x0.64mm_HandSolder
- R16: renamed from R25; footprint (none) -> Resistor_SMD:R_0402_1005Metric_Pad0.72x0.64mm_HandSolder
- R17: renamed from R43; footprint (none) -> Resistor_SMD:R_0402_1005Metric_Pad0.72x0.64mm_HandSolder
- R18: renamed from R26; footprint (none) -> Resistor_SMD:R_0402_1005Metric_Pad0.72x0.64mm_HandSolder
- R19: renamed from R44; footprint (none) -> Resistor_SMD:R_0402_1005Metric_Pad0.72x0.64mm_HandSolder
- R2: renamed from R36; footprint (none) -> Resistor_SMD:R_0402_1005Metric_Pad0.72x0.64mm_HandSolder
- R20: renamed from R27; footprint (none) -> Resistor_SMD:R_0402_1005Metric_Pad0.72x0.64mm_HandSolder
- R21: renamed from R45; footprint (none) -> Resistor_SMD:R_0402_1005Metric_Pad0.72x0.64mm_HandSolder
- R22: renamed from R28; footprint (none) -> Resistor_SMD:R_0402_1005Metric_Pad0.72x0.64mm_HandSolder
- R23: renamed from R46; footprint (none) -> Resistor_SMD:R_0402_1005Metric_Pad0.72x0.64mm_HandSolder
- R24: renamed from R29; footprint (none) -> Resistor_SMD:R_0402_1005Metric_Pad0.72x0.64mm_HandSolder
- R25: renamed from R47; footprint (none) -> Resistor_SMD:R_0402_1005Metric_Pad0.72x0.64mm_HandSolder
- R26: renamed from R30; footprint (none) -> Resistor_SMD:R_0402_1005Metric_Pad0.72x0.64mm_HandSolder
- R27: renamed from R48; footprint (none) -> Resistor_SMD:R_0402_1005Metric_Pad0.72x0.64mm_HandSolder
- R28: renamed from R31; footprint (none) -> Resistor_SMD:R_0402_1005Metric_Pad0.72x0.64mm_HandSolder
- R29: renamed from R49; footprint (none) -> Resistor_SMD:R_0402_1005Metric_Pad0.72x0.64mm_HandSolder
- R3: renamed from R18; footprint (none) -> Resistor_SMD:R_0402_1005Metric_Pad0.72x0.64mm_HandSolder
- R30: renamed from R32; footprint (none) -> Resistor_SMD:R_0402_1005Metric_Pad0.72x0.64mm_HandSolder
- R31: renamed from R50; footprint (none) -> Resistor_SMD:R_0402_1005Metric_Pad0.72x0.64mm_HandSolder
- R32: renamed from R33; footprint (none) -> Resistor_SMD:R_0402_1005Metric_Pad0.72x0.64mm_HandSolder
- R33: renamed from R51; footprint (none) -> Resistor_SMD:R_0402_1005Metric_Pad0.72x0.64mm_HandSolder
- R34: footprint (none) -> Resistor_SMD:R_0402_1005Metric_Pad0.72x0.64mm_HandSolder
- R35: renamed from R52; footprint (none) -> Resistor_SMD:R_0402_1005Metric_Pad0.72x0.64mm_HandSolder
- R36: renamed from R35; footprint (none) -> Resistor_SMD:R_0402_1005Metric_Pad0.72x0.64mm_HandSolder
- R37: renamed from R53; footprint (none) -> Resistor_SMD:R_0402_1005Metric_Pad0.72x0.64mm_HandSolder
- R38: renamed from R54; footprint (none) -> Resistor_SMD:R_0402_1005Metric_Pad0.72x0.64mm_HandSolder
- R39: renamed from R55; footprint (none) -> Resistor_SMD:R_0402_1005Metric_Pad0.72x0.64mm_HandSolder
- R4: renamed from R37; footprint (none) -> Resistor_SMD:R_0402_1005Metric_Pad0.72x0.64mm_HandSolder
- R40: renamed from R2; footprint (none) -> Resistor_SMD:R_0402_1005Metric_Pad0.72x0.64mm_HandSolder
- R5: renamed from R20; footprint (none) -> Resistor_SMD:R_0402_1005Metric_Pad0.72x0.64mm_HandSolder
- R6: renamed from R38; footprint (none) -> Resistor_SMD:R_0402_1005Metric_Pad0.72x0.64mm_HandSolder
- R7: renamed from R21; footprint (none) -> Resistor_SMD:R_0402_1005Metric_Pad0.72x0.64mm_HandSolder
- R8: renamed from R39; footprint (none) -> Resistor_SMD:R_0402_1005Metric_Pad0.72x0.64mm_HandSolder
- R9: renamed from R22; footprint (none) -> Resistor_SMD:R_0402_1005Metric_Pad0.72x0.64mm_HandSolder
- renumbered J3 to J16, J7 to J2, J8 to J3, Q2 to Q1, Q14 to Q10, Q6 to Q11, Q15 to Q12, Q7 to Q13, Q16 to Q14, Q8 to Q15, Q17 to Q16, Q9 to Q17, Q10 to Q2, Q1 to Q3, Q11 to Q4, Q3 to Q5, Q12 to Q6, Q4 to Q7, Q13 to Q8, Q5 to Q9, SW2 to SW1, SW1 to SW2, U3 to U2, U6 to U3, U2 to U5
Connections:
- net V_LIDAR2 is gone; now on net I2C1_SCL: Q20.3 (D)
- net +3.3V: now also J12.3 (Pin_3), R45.2, R47.2
- net +5V: now also J12.1 (Pin_1), R46.2, R48.2; no longer C25.2, C26.2, C27.2, C28.2, C29.2, C30.2, C31.2, C32.2, IC1.5 (VM), IC2.5 (VM), IC3.5 (VM), IC4.5 (VM)
- net ADC1/14: now also IC1.1 (IPROPI), R42.2
- net ADC1/15: now also IC2.1 (IPROPI), R43.2
- net ADC1/7: now also IC4.1 (IPROPI), R41.2
- net ADC1/9: now also IC3.1 (IPROPI), R44.2
- net GND: now also J4.5 (Pin_5), J5.5 (Pin_5), J6.5 (Pin_5), J7.5 (Pin_5), R41.1, R42.1, R43.1, R44.1
- net I2C1_SCL: now also R47.1; no longer Q20.2 (S)
- net I2C1_SDA: now also R45.1; no longer Q19.2 (S)
- net I2C3_SCL: now also Q20.2 (S), R48.1
- net I2C3_SDA: now also Q19.2 (S), R46.1
- net V_M1A: now also J8.1 (Pin_1); no longer J9.1 (Pin_1)
- net V_M1B: now also J8.2 (Pin_2); no longer J9.2 (Pin_2)
- net V_M2A: now also J9.1 (Pin_1); no longer J10.1 (Pin_1)
- net V_M2B: now also J9.2 (Pin_2); no longer J10.2 (Pin_2)
- net V_M3A: now also J10.1 (Pin_1); no longer J11.1 (Pin_1)
- net V_M3B: now also J10.2 (Pin_2); no longer J11.2 (Pin_2)
- net V_M4A: now also J11.1 (Pin_1)
- net V_M4B: now also J11.2 (Pin_2)
- net Mtr1_EncoderZ: now reaches CN2.14 (Pin_14)
- net Mtr1_EncoderZ: now also J4.4 (Pin_4)
- net Mtr1_EncoderA: now reaches CN2.2 (Pin_2)
- net Mtr1_EncoderA: now also J4.2 (Pin_2)
- net Mtr2_EncoderA: now reaches CN2.22 (Pin_22)
- net Mtr2_EncoderA: now also J5.2 (Pin_2)
- net Mtr2_EncoderB: now reaches CN2.26 (Pin_26)
- net Mtr2_EncoderB: now also J5.3 (Pin_3)
- net Mtr3_EncoderZ: now reaches CN2.27 (Pin_27)
- net Mtr3_EncoderZ: now also J6.4 (Pin_4)
- net Mtr2_EncoderZ: now reaches CN2.28 (Pin_28)
- net Mtr2_EncoderZ: now also J5.4 (Pin_4)
- net Mtr3_EncoderB: now reaches CN2.31 (Pin_31)
- net Mtr3_EncoderB: now also J6.3 (Pin_3)
- net Mtr3_EncoderA: now reaches CN2.33 (Pin_33)
- net Mtr3_EncoderA: now also J6.2 (Pin_2)
- net Mtr1_EncoderB: now reaches CN2.4 (Pin_4)
- net Mtr1_EncoderB: now also J4.3 (Pin_3)
- net Mtr4_EncoderA: now reaches CN1.17 (Pin_17)
- net Mtr4_EncoderA: now also J7.2 (Pin_2)
- net Mtr4_EncoderB: now reaches CN1.21 (Pin_21)
- net Mtr4_EncoderB: now also J7.3 (Pin_3)
- net Mtr4_EncoderZ: now reaches CN1.23 (Pin_23)
- net Mtr4_EncoderZ: now also J7.4 (Pin_4)
- new net V_DCMTR: C25.2, C26.2, C27.2, C28.2, C29.2, C30.2, C31.2, C32.2, IC1.5 (VM), IC2.5 (VM), IC3.5 (VM), IC4.5 (VM)
- new net V_encoder: J12.2 (Pin_2), J4.1 (Pin_1), J5.1 (Pin_1), J6.1 (Pin_1), J7.1 (Pin_1)
- no-connect marks 12 -> 56
Other:
- note added: "18 Servo Header"
- note added: "Encoder Connectors"
- note added: "Encoder Select Voltage"
- note added: "Header pins, use shunt to select voltage"
- note added: "I2C Add: 0x62"
- note added: "I2C Add: 0x68"
- note added: "I2C Add: 0x69"
- note added: "Motor Connectors"
- note added: "Power Connectors"
- note removed: "Motor Terminals"
- note removed: "Power Terminals"
- note removed: "Servo Header"
- moved on the sheet: C1, C10, C11, C12, C13, C14, C15, C16, C17, C18, C19, C2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

Commit message: Added Arduino connectors and LEDs. Changed servo footprint and power in labels.
Parts:
- removed J13, J14, J17: Conn_01x12_seperated, Connector_PinHeader_1.00mm:PinHeader_1x12_P1.00mm_Vertical_SMD_Pin1Right, symbol Connector:Conn_01x03_Pin
- removed J15: Conn_01x12_seperated, Connector_PinHeader_1.00mm:PinHeader_1x06_P1.00mm_Vertical_SMD_Pin1Left, symbol Connector:Conn_01x03_Pin
- removed J16: Conn_01x12_seperated, symbol Connector:Conn_01x03_Pin
- added D1: Red LED, symbol Device:LED
- added D2, D3, D4: Yellow LED, symbol Device:LED
- added J13, J14, J15, J16, J17, J18, J19, J20, J21, J22, J23, J24, J25, J26, J27, J28, J29, J30: Conn_01x03, Connector_PinHeader_2.54mm:PinHeader_1x03_P2.54mm_Vertical, symbol Connector_Generic:Conn_01x03
- added J31: Conn_01x06, symbol Connector_Generic:Conn_01x06
- added J32, J33: Conn_01x08, symbol Connector_Generic:Conn_01x08
- added J34: Conn_01x10, symbol Connector_Generic:Conn_01x10
- added R49, R50, R51, R52: 100, Resistor_SMD:R_0402_1005Metric_Pad0.72x0.64mm_HandSolder, symbol Device:R
- J8: renamed from J12; footprint Connector_PinHeader_1.00mm:PinHeader_1x03_P1.00mm_Vertical_SMD_Pin1Left -> Connector_PinHeader_2.54mm:PinHeader_1x03_P2.54mm_Vertical
- renumbered J9 to J10, J10 to J11, J11 to J12, J8 to J9, R45 to R41, R46 to R42, R47 to R43, R48 to R44, R41 to R45, R42 to R46, R43 to R47, R44 to R48
Connections:
- net V_DCMotor is gone; now on net V_DCMTR: C14.1, J3.1 (Pin_1)
- net +3.3V: now also D1.2 (A), J33.4 (Pin_4)
- net +5V: now also D2.2 (A), J33.5 (Pin_5)
- net ADC1/7: now also J34.4 (Pin_4)
- net GND: now also J25.1 (Pin_1), J25.2 (Pin_2), J25.3 (Pin_3), J26.1 (Pin_1), J26.2 (Pin_2), J26.3 (Pin_3), J27.1 (Pin_1), J27.2 (Pin_2), J27.3 (Pin_3), J28.1 (Pin_1), J28.2 (Pin_2), J28.3 (Pin_3), J29.1 (Pin_1), J29.2 (Pin_2), J29.3 (Pin_3), J30.1 (Pin_1), J30.2 (Pin_2), J30.3 (Pin_3), J33.6 (Pin_6), J33.7 (Pin_7), R49.2, R50.2, R51.2, R52.2
- net I2C1_SCL: now also J34.10 (Pin_10)
- net I2C1_SDA: now also J34.9 (Pin_9)
- net Mtr3_EncoderA: now also J32.3 (Pin_3)
- net Mtr3_EncoderB: now also J32.4 (Pin_4)
- net Mtr3_EncoderZ: now also J32.6 (Pin_6)
- net PWM1/1: now also J32.8 (Pin_8)
- net PWM1/2: now also J34.1 (Pin_1)
- net PWM2/1: now also J34.6 (Pin_6)
- net PWM2/3: now also J32.7 (Pin_7)
- net PWM3/1: now also J34.5 (Pin_5)
- net PWM3/2: now also J32.5 (Pin_5), J34.2 (Pin_2)
- net PWM4/1: now also J34.3 (Pin_3)
- net V_DCMTR: now also D4.2 (A)
- net V_Servo: now also D3.2 (A), J19.1 (Pin_1), J19.2 (Pin_2), J19.3 (Pin_3), J20.1 (Pin_1), J20.2 (Pin_2), J20.3 (Pin_3), J21.1 (Pin_1), J21.2 (Pin_2), J21.3 (Pin_3), J22.1 (Pin_1), J22.2 (Pin_2), J22.3 (Pin_3), J23.1 (Pin_1), J23.2 (Pin_2), J23.3 (Pin_3), J24.1 (Pin_1), J24.2 (Pin_2), J24.3 (Pin_3)
- net V_Servo1: now also J13.1 (Pin_1)
- net V_Servo10: now also J16.1 (Pin_1)
- net V_Servo11: now also J16.2 (Pin_2)
- net V_Servo12: now also J16.3 (Pin_3)
- net V_Servo13: now also J17.1 (Pin_1)
- net V_Servo14: now also J17.2 (Pin_2)
- net V_Servo15: now also J17.3 (Pin_3)
- net V_Servo16: now also J18.1 (Pin_1)
- net V_Servo17: now also J18.2 (Pin_2)
- net V_Servo18: now also J18.3 (Pin_3)
- net V_Servo2: now also J13.2 (Pin_2)
- net V_Servo3: now also J13.3 (Pin_3)
- net V_Servo4: now also J14.1 (Pin_1)
- net V_Servo5: now also J14.2 (Pin_2)
- net V_Servo6: now also J14.3 (Pin_3)
- net V_Servo7: now also J15.1 (Pin_1)
- net V_Servo8: now also J15.2 (Pin_2)
- net V_Servo9: now also J15.3 (Pin_3)
- net at CN2.35 (Pin_35): now also J32.2 (Pin_2)
- net at CN2.37 (Pin_37): now also J32.1 (Pin_1)
- net at CN2.7 (Pin_7): now also J34.8 (Pin_8)
- net at CN2.9 (Pin_9): now also J34.7 (Pin_7)
- net at CN1.24 (Pin_24): now also J33.8 (Pin_8)
- new net: D1.1 (K), R49.1
- new net: D3.1 (K), R51.1
- new net: D2.1 (K), R50.1
- new net: D4.1 (K), R52.1
- no-connect marks 56 -> 50
Other:
- note added: "18 Servo"
- note added: "LEDs"
- note added: "Morpho and Arduino Header"
- note added: "Servo Headers"
- note removed: "18 Servo Header"
- note removed: "Morpho Header"
- moved on the sheet: C10, C11, C12, C13, C14, C15, C16, C17, C18, C19, C20, C21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

Commit message: Started PCB, alligned and placed microcontroller components
Parts:
- removed D3, D4: Yellow LED, symbol Device:LED
- removed R51, R52: 100, Resistor_SMD:R_0402_1005Metric_Pad0.72x0.64mm_HandSolder, symbol Device:R
- removed SW2: SW_SPDT, symbol Switch:SW_SPDT
- added J6: Conn_01x03, Connector_PinHeader_2.54mm:PinHeader_1x03_P2.54mm_Vertical_SMD_Pin1Left, symbol Connector_Generic:Conn_01x03
- CN1: renamed from CN2; footprint Connector_PinSocket_2.54mm:PinSocket_2x19_P2.54mm_Vertical -> Connector_PinHeader_2.54mm:PinHeader_1x38_P2.54mm_Vertical
- CN2: renamed from CN1; footprint Connector_PinSocket_2.54mm:PinSocket_2x19_P2.54mm_Vertical -> Connector_PinHeader_2.54mm:PinHeader_1x38_P2.54mm_Vertical
- D1: renamed from D2; footprint (none) -> LED_SMD:LED_0402_1005Metric_Pad0.77x0.64mm_HandSolder
- D2: renamed from D1; footprint (none) -> LED_SMD:LED_0402_1005Metric_Pad0.77x0.64mm_HandSolder
- J11: renamed from J34; footprint (none) -> Connector_PinHeader_2.54mm:PinHeader_1x10_P2.54mm_Vertical_SMD_Pin1Left
- J12: renamed from J33; footprint (none) -> Connector_PinHeader_2.54mm:PinHeader_1x08_P2.54mm_Vertical_SMD_Pin1Left
- J14: renamed from J31; footprint (none) -> Connector_PinHeader_2.54mm:PinHeader_1x06_P2.54mm_Vertical_SMD_Pin1Left
- J15: renamed from J32; footprint (none) -> Connector_PinHeader_2.54mm:PinHeader_1x08_P2.54mm_Vertical_SMD_Pin1Right
- J18: renamed from J13; footprint Connector_PinHeader_2.54mm:PinHeader_1x03_P2.54mm_Vertical -> Connector_PinHeader_2.54mm:PinHeader_1x03_P2.54mm_Vertical_SMD_Pin1Left
- J21: renamed from J14; footprint Connector_PinHeader_2.54mm:PinHeader_1x03_P2.54mm_Vertical -> Connector_PinHeader_2.54mm:PinHeader_1x03_P2.54mm_Vertical_SMD_Pin1Left
- J24: renamed from J15; footprint Connector_PinHeader_2.54mm:PinHeader_1x03_P2.54mm_Vertical -> Connector_PinHeader_2.54mm:PinHeader_1x03_P2.54mm_Vertical_SMD_Pin1Left
- J27: renamed from J16; footprint Connector_PinHeader_2.54mm:PinHeader_1x03_P2.54mm_Vertical -> Connector_PinHeader_2.54mm:PinHeader_1x03_P2.54mm_Vertical_SMD_Pin1Left
- J30: renamed from J17; footprint Connector_PinHeader_2.54mm:PinHeader_1x03_P2.54mm_Vertical -> Connector_PinHeader_2.54mm:PinHeader_1x03_P2.54mm_Vertical_SMD_Pin1Left
- J33: renamed from J18; footprint Connector_PinHeader_2.54mm:PinHeader_1x03_P2.54mm_Vertical -> Connector_PinHeader_2.54mm:PinHeader_1x03_P2.54mm_Vertical_SMD_Pin1Left
- J4: renamed from J1; footprint Connector_PinHeader_1.00mm:PinHeader_1x04_P1.00mm_Vertical_SMD_Pin1Left -> Connector_PinHeader_2.54mm:PinHeader_1x04_P2.54mm_Vertical_SMD_Pin1Left
- LiDAR-V1: footprint (none) -> Connector_PinHeader_2.54mm:PinHeader_1x05_P2.54mm_Vertical_SMD_Pin1Left
- SW1: footprint (none) -> Button_Switch_SMD:SW_DIP_SPSTx02_Slide_6.7x6.64mm_W8.61mm_P2.54mm_LowProfile
- Y1: footprint (none) -> Crystal:Crystal_SMD_2016-4Pin_2.0x1.6mm
- renumbered C29 to C10, C3 to C11, C5 to C12, C7 to C13, C11 to C14, C18 to C15, C26 to C16, C30 to C17, C17 to C18, C14 to C19, C27 to C20, C31 to C21, C12 to C22, C15 to C23, C19 to C24, C21 to C25, C28 to C26, C32 to C27, C13 to C28, C16 to C29, C4 to C3, C20 to C30, C22 to C31, C24 to C32, C6 to C4, C8 to C5, C9 to C6, C10 to C7, C23 to C8, C25 to C9, J4 to J1, J11 to J10, J7 to J13, J12 to J16, J8 to J17, J9 to J2, J25 to J20, J20 to J22, J26 to J23, J21 to J25, J27 to J26, J22 to J28, J28 to J29, J5 to J3, J23 to J31, J29 to J32, J24 to J34, J30 to J35, J10 to J5, J2 to J7, J3 to J8, J6 to J9, Q19 to Q1, Q15 to Q10, Q17 to Q11, Q2 to Q12, Q4 to Q13, Q6 to Q14, Q8 to Q15, Q10 to Q16, Q12 to Q17, Q14 to Q18, Q16 to Q19, Q20 to Q2, Q18 to Q20, Q1 to Q3, Q3 to Q4, Q7 to Q6, Q9 to Q7, Q11 to Q8, Q13 to Q9, R46 to R1, R45 to R10, R41 to R11, R43 to R12, R1 to R13, R5 to R14, R9 to R15, R14 to R16, R18 to R17, R22 to R18, R26 to R19, R40 to R2, R30 to R20, R34 to R21, R42 to R22, R44 to R23, R3 to R24, R7 to R25, R11 to R26, R16 to R27, R20 to R28, R24 to R29, R47 to R3, R28 to R30, R32 to R31, R36 to R32, R2 to R33, R6 to R34, R10 to R35, R15 to R36, R19 to R37, R23 to R38, R27 to R39, R13 to R4, R31 to R40, R35 to R41, R4 to R42, R8 to R43, R12 to R44, R17 to R45, R21 to R46, R25 to R47, R29 to R48, R33 to R49, R50 to R5, R37 to R50, R49 to R6, R48 to R7, R38 to R8, R39 to R9, U2 to U1, U1 to U2
Connections:
- net +3.3V: now also J6.1 (Pin_1)
- net BOOT0: now also R4.1, J6.2 (Pin_2)
- net GND: now also J6.3 (Pin_3)
- net PWM1/1: no longer CN1.23 (Pin_23), J15.8 (Pin_8)
- net PWM1/2: no longer CN1.21 (Pin_21), J11.1 (Pin_1)
- net PWM2/1: now also CN2.28 (Pin_28), J14.1 (Pin_1); no longer CN1.11 (Pin_11), IC1.2 (IN2), IC2.2 (IN2), IC3.2 (IN2), IC4.2 (IN2), J11.6 (Pin_6)
- net PWM2/2: now also CN2.30 (Pin_30), J14.2 (Pin_2)
- net PWM2/3: no longer CN1.25 (Pin_25), J15.7 (Pin_7)
- net PWM3/1: no longer CN1.13 (Pin_13), IC1.3 (IN1), IC2.3 (IN1), IC3.3 (IN1), IC4.3 (IN1), J11.5 (Pin_5)
- net PWM3/2: no longer CN1.19 (Pin_19), CN1.29 (Pin_29), J11.2 (Pin_2), J15.5 (Pin_5)
- net PWM4/1: no longer CN1.17 (Pin_17), J11.3 (Pin_3)
- net at J14.3 (Pin_3): now also CN2.32 (Pin_32)
- net PWM1/2N: now reaches J14.4 (Pin_4)
- net PWM1/2N: now also CN2.34 (Pin_34)
- net at J14.5 (Pin_5): now also CN2.36 (Pin_36)
- net at J14.6 (Pin_6): now also CN2.38 (Pin_38)
- new net PWM1/1_M3: CN1.23 (Pin_23), IC3.3 (IN1), J15.8 (Pin_8)
- new net PWM1/2_M3: CN1.21 (Pin_21), IC3.2 (IN2), J11.1 (Pin_1)
- new net PWM2/1_M1: CN1.11 (Pin_11), IC1.2 (IN2), J11.6 (Pin_6)
- new net PWM2/3_M4: CN1.25 (Pin_25), IC4.2 (IN2), J15.7 (Pin_7)
- new net PWM3/1_M1: CN1.13 (Pin_13), IC1.3 (IN1), J11.5 (Pin_5)
- new net PWM3/2_M2: CN1.19 (Pin_19), IC2.3 (IN1), J11.2 (Pin_2)
- new net PWM3/2_M4: CN1.29 (Pin_29), IC4.3 (IN1), J15.5 (Pin_5)
- new net PWM4/1_M2: CN1.17 (Pin_17), IC2.2 (IN2), J11.3 (Pin_3)
- no-connect marks 50 -> 44
Other:
- note added: "BOOT Select Voltage"
- moved on the sheet: D1, D2, R4, R5, R6
