File: DAWG_ServoDriver.kicad_sch (KiCad schematic)
At the start: 154 parts, among them CN1 Conn_02x19_Odd_Even, CN2 Conn_02x19_Odd_Even, IC1 DRV8251ADDAR, IC2 DRV8251ADDAR, IC3 DRV8251ADDAR, IC4 DRV8251ADDAR, J1 Conn_01x05, J10 Screw_Terminal_01x02, J11 Conn_01x10, J12 Conn_01x08, J13 Conn_01x05, J14 Conn_01x06, J15 Conn_01x08, J16 Screw_Terminal_01x02, J17 Conn_01x03, J18 Conn_01x03, J19 Conn_01x03, J2 Screw_Terminal_01x02, J20 Conn_01x03, J21 Conn_01x03, J22 Conn_01x03, J23 Conn_01x03, J24 Conn_01x03, J25 Conn_01x03, J26 Conn_01x03, J27 Conn_01x03, J28 Conn_01x03, J29 Conn_01x03, J3 Conn_01x05, J30 Conn_01x03, J31 Conn_01x03, J32 Conn_01x03, J33 Conn_01x03, J34 Conn_01x03, J35 Conn_01x03, J4 Conn_01x04_Pin, J5 Screw_Terminal_01x02, J6 Conn_01x03, J7 Screw_Terminal_01x02, J8 Screw_Terminal_01x02, J9 Conn_01x05, Q1 BSS138, Q10 BSS138, Q11 BSS138, Q12 BSS138, Q13 BSS138, Q14 BSS138, Q15 BSS138, Q16 BSS138, Q17 BSS138, Q18 BSS138, Q19 BSS138, Q2 BSS138, Q20 BSS138, Q3 BSS138, Q4 BSS138, Q5 BSS138, Q6 BSS138, Q7 BSS138, Q8 BSS138, Q9 BSS138, SW1 SW_Push, U1 TPS62177DQC, U2 STM32G431C8Tx, U3 LD1117S12TR_SOT223, U4 ICM-20602, U5 ICM-20602, Y1 Crystal_GND24

Commit message: Placed mos most components, routed servo.
Parts:
- added IC5: ESP32-PICO-MINI-02-N8R2, ESP32PICOMINI02N8R2, symbol MCU_Espressif:ESP32-PICO-MINI-02-N8R2
- added J36: Conn_01x03, Connector_PinHeader_2.54mm:PinHeader_1x03_P2.54mm_Vertical, symbol Connector_Generic:Conn_01x03
- CN10: renamed from CN1; footprint Connector_PinHeader_2.54mm:PinHeader_1x38_P2.54mm_Vertical -> Connector_PinHeader_2.54mm:PinHeader_2x19_P2.54mm_Vertical
- CN7: renamed from CN2; footprint Connector_PinHeader_2.54mm:PinHeader_1x38_P2.54mm_Vertical -> Connector_PinHeader_2.54mm:PinHeader_2x19_P2.54mm_Vertical
- J1, J13, J3, J9: footprint TerminalBlock_MetzConnect:TerminalBlock_MetzConnect_Type011_RT05505HBWC_1x05_P5.00mm_Horizontal -> Connector_PinHeader_2.54mm:PinHeader_1x05_P2.54mm_Vertical
- J10, J16, J2, J5: footprint TerminalBlock_MetzConnect:TerminalBlock_MetzConnect_Type011_RT05502HBWC_1x02_P5.00mm_Horizontal -> Connector_PinHeader_2.54mm:PinHeader_1x02_P2.54mm_Vertical
- J11: footprint Connector_PinHeader_2.54mm:PinHeader_1x10_P2.54mm_Vertical_SMD_Pin1Left -> Connector_PinHeader_2.54mm:PinHeader_1x10_P2.54mm_Vertical
- J12: footprint Connector_PinHeader_2.54mm:PinHeader_1x08_P2.54mm_Vertical_SMD_Pin1Left -> Connector_PinHeader_2.54mm:PinHeader_1x08_P2.54mm_Vertical
- J14: footprint Connector_PinHeader_2.54mm:PinHeader_1x06_P2.54mm_Vertical_SMD_Pin1Left -> Connector_PinHeader_2.54mm:PinHeader_1x06_P2.54mm_Vertical
- J15: footprint Connector_PinHeader_2.54mm:PinHeader_1x08_P2.54mm_Vertical_SMD_Pin1Right -> Connector_PinHeader_2.54mm:PinHeader_1x08_P2.54mm_Vertical
- J18, J21, J24, J27, J30, J33, J6: footprint Connector_PinHeader_2.54mm:PinHeader_1x03_P2.54mm_Vertical_SMD_Pin1Left -> Connector_PinHeader_2.54mm:PinHeader_1x03_P2.54mm_Vertical
- J4: footprint Connector_PinHeader_2.54mm:PinHeader_1x04_P2.54mm_Vertical_SMD_Pin1Left -> Connector_PinHeader_2.54mm:PinHeader_1x04_P2.54mm_Vertical
- LiDAR-V1: footprint Connector_PinHeader_2.54mm:PinHeader_1x05_P2.54mm_Vertical_SMD_Pin1Left -> Connector_PinHeader_2.54mm:PinHeader_1x05_P2.54mm_Vertical
- SW1: footprint Button_Switch_SMD:SW_DIP_SPSTx02_Slide_6.7x6.64mm_W8.61mm_P2.54mm_LowProfile -> Button_Switch_SMD:SW_Push_1P1T-SH_NO_CK_KMR2xxG
Connections:
- net PWM1/2N is gone; now on net IsenseM4: CN7.34 (Pin_34), J14.4 (Pin_4)
- net +BATT: now also J36.2 (Pin_2)
- net GND: now also CN10.9 (Pin_9), J11.7 (Pin_7), IC5.36 (GND_5), IC5.37 (GND_6), IC5.38 (GND_7), IC5.39 (GND_8), IC5.40 (GND_9), IC5.41 (GND_10), IC5.42 (GND_11), IC5.43 (GND_12), IC5.44 (GND_13), IC5.45 (GND_14), IC5.46 (GND_15), IC5.47 (GND_16), IC5.48 (GND_17), IC5.49 (GND_18), IC5.50 (GND_19), IC5.51 (GND_20), IC5.52 (GND_21), IC5.53 (GND_22), IC5.54 (GND_23), IC5.55 (GND_24), IC5.56 (GND_25), IC5.57 (GND_26), IC5.58 (GND_27), IC5.59 (GND_28), IC5.60 (GND_29), IC5.61 (GND_30)
- net I2C3_SCL: no longer U2.30 (PA8)
- net IMU1_INT: now also CN10.37 (Pin_37), J15.1 (Pin_1); no longer CN10.12 (Pin_12)
- net IMU2_INT: now also CN10.35 (Pin_35), J15.2 (Pin_2); no longer CN10.16 (Pin_16)
- net Mtr1_EncoderA: now also CN10.11 (Pin_11), J11.6 (Pin_6); no longer CN10.2 (Pin_2)
- net Mtr1_EncoderB: now also CN10.17 (Pin_17), J11.3 (Pin_3); no longer CN10.4 (Pin_4)
- net Mtr1_EncoderZ: now also CN10.16 (Pin_16); no longer CN10.14 (Pin_14)
- net Mtr2_EncoderA: now also CN10.29 (Pin_29), J15.5 (Pin_5); no longer CN10.22 (Pin_22)
- net Mtr2_EncoderB: now also CN10.31 (Pin_31), J15.4 (Pin_4); no longer CN10.26 (Pin_26)
- net Mtr2_EncoderZ: no longer CN10.28 (Pin_28)
- net Mtr3_EncoderA: no longer CN10.33 (Pin_33), J15.3 (Pin_3)
- net Mtr3_EncoderB: no longer CN10.31 (Pin_31), J15.4 (Pin_4)
- net Mtr3_EncoderZ: no longer CN10.27 (Pin_27), J15.6 (Pin_6)
- net PWM15/1: now also Q12.2 (S), R42.1; no longer Q18.2 (S), R48.1
- net PWM15/2: now also Q11.2 (S), R32.1, U2.29 (PB15); no longer Q19.2 (S), R49.1, U2.11 (PA3)
- net PWM16/1: now also Q5.2 (S), R26.1; no longer Q20.2 (S), R50.1
- net PWM1/1: now also Q10.2 (S), R31.1, U2.30 (PA8); no longer Q3.2 (S), R24.1, U2.15 (PA7)
- net PWM1/1_M3: no longer CN10.23 (Pin_23), J15.8 (Pin_8)
- net PWM1/2: now also Q9.2 (S), R30.1; no longer Q4.2 (S), R25.1
- net PWM1/2_M3: no longer CN10.21 (Pin_21), J11.1 (Pin_1)
- net PWM1/3: now also Q8.2 (S), R29.1; no longer Q5.2 (S), R26.1
- net PWM1/4: now also Q7.2 (S), R28.1; no longer Q6.2 (S), R27.1
- net PWM2/1: no longer CN7.28 (Pin_28), J14.1 (Pin_1), Q7.2 (S), R28.1
- net PWM2/1_M1: now also CN10.13 (Pin_13), J11.5 (Pin_5); no longer CN10.11 (Pin_11), J11.6 (Pin_6)
- net PWM2/2: no longer CN7.30 (Pin_30), J14.2 (Pin_2), Q8.2 (S), R29.1
- net PWM2/3: no longer Q9.2 (S), R30.1
- net PWM2/3_M4: no longer CN10.25 (Pin_25), J15.7 (Pin_7)
- net PWM2/4: no longer Q10.2 (S), R31.1
- net PWM3/1: now also Q16.2 (S), R46.1; no longer Q11.2 (S), R32.1
- net PWM3/1_M1: now also CN10.15 (Pin_15), J11.4 (Pin_4); no longer CN10.13 (Pin_13), J11.5 (Pin_5)
- net PWM3/2: now also Q15.2 (S), R45.1; no longer Q12.2 (S), R42.1
- net PWM3/2_M4: no longer CN10.29 (Pin_29), J15.5 (Pin_5)
- net PWM3/3: now also Q14.2 (S), R44.1; no longer Q13.2 (S), R43.1
- net PWM3/4: now also Q13.2 (S), R43.1; no longer Q14.2 (S), R44.1
- net PWM4/1: now also Q4.2 (S), R25.1; no longer Q15.2 (S), R45.1
- net PWM4/1_M2: now also CN10.27 (Pin_27), J15.6 (Pin_6); no longer CN10.17 (Pin_17), J11.3 (Pin_3)
- net PWM4/2: now also Q6.2 (S), R27.1; no longer Q16.2 (S), R46.1
- net PWM4/4: now also Q3.2 (S), R24.1; no longer Q17.2 (S), R47.1
- net V_DCMTR: now also J36.1 (Pin_1)
- net V_Servo: now also J36.3 (Pin_3)
- net IsenseM3: now reaches CN7.32 (Pin_32), J14.3 (Pin_3)
- net IsenseM3: now also IC3.1 (IPROPI), R7.2
- net ADC1/14 renamed IsenseM1
- net IsenseM1: now also CN7.28 (Pin_28), J14.1 (Pin_1); no longer CN10.34 (Pin_34)
- net ADC1/15 renamed IsenseM2
- net IsenseM2: now also CN7.30 (Pin_30), J14.2 (Pin_2); no longer CN10.6 (Pin_6)
- net ADC1/7 renamed IsenseM4
- net IsenseM4: no longer CN10.15 (Pin_15), J11.4 (Pin_4)
- removed net ADC1/9: CN10.24 (Pin_24), IC3.1 (IPROPI), R7.2
- new net: Q17.2 (S), R47.1
- new net: Q18.2 (S), R48.1
- new net: Q20.2 (S), R50.1
- new net: CN10.21 (Pin_21), J11.1 (Pin_1)
- new net: CN10.23 (Pin_23), J15.8 (Pin_8)
- new net: CN10.25 (Pin_25), J15.7 (Pin_7)
- new net: CN10.33 (Pin_33), J15.3 (Pin_3)
- new net: Q19.2 (S), R49.1
- no-connect marks 44 -> 43
Other:
- note added: "ESP32-PICO-MINI-02"
- moved on the sheet: C18, C19, CN7, D1, D2, J12, J14, J7, J8, R5, R6
