File: DAWG_ServoDriver.kicad_sch (KiCad schematic)
At the start: 154 parts, among them CN10 Conn_02x19_Odd_Even, CN7 Conn_02x19_Odd_Even, IC1 DRV8251ADDAR, IC2 DRV8251ADDAR, IC3 DRV8251ADDAR, IC4 DRV8251ADDAR, IC5 ESP32-PICO-MINI-02-N8R2, J1 Screw_Terminal_01x06, J11 Conn_01x10, J12 Conn_01x08, J13 Screw_Terminal_01x06, J14 Conn_01x06, J15 Conn_01x08, J17 Conn_01x03, J18 Conn_01x03, J19 Conn_01x03, J2 Conn_01x04, J20 Conn_01x03, J21 Conn_01x03, J22 Conn_01x03, J23 Conn_01x03, J24 Conn_01x03, J25 Conn_01x03, J26 Conn_01x03, J27 Conn_01x03, J28 Conn_01x03, J29 Conn_01x03, J3 Screw_Terminal_01x06, J30 Conn_01x03, J31 Conn_01x03, J32 Conn_01x03, J33 Conn_01x03, J34 Conn_01x03, J35 Conn_01x03, J36 Conn_01x03, J4 Conn_01x04_Pin, J5 Conn_01x04, J6 Conn_01x03, J7 Screw_Terminal_01x02, J8 Screw_Terminal_01x02, J9 Screw_Terminal_01x06, Q1 BSS138, Q10 BSS138, Q11 BSS138, Q12 BSS138, Q13 BSS138, Q14 BSS138, Q15 BSS138, Q16 BSS138, Q17 BSS138, Q18 BSS138, Q19 BSS138, Q2 BSS138, Q20 BSS138, Q3 BSS138, Q4 BSS138, Q5 BSS138, Q6 BSS138, Q7 BSS138, Q8 BSS138, Q9 BSS138, SW1 SW_Push, U1 TPS62177DQC, U2 STM32G431C8Tx, U3 LD1117S12TR_SOT223, U4 ICM-20602, U5 ICM-20602, Y1 Crystal_GND24

Commit message: added esp32 & lidar, finished routing unrouted stuff
Parts:
- removed J2, J5: Conn_01x04, symbol Connector_Generic:Conn_01x04
- added C33: 100n, Capacitor_SMD:C_0402_1005Metric_Pad0.74x0.62mm_HandSolder, symbol Device:C
- added C34: 22u, Capacitor_SMD:C_0402_1005Metric_Pad0.74x0.62mm_HandSolder, symbol Device:C
- added C35: 1u, Capacitor_SMD:C_0402_1005Metric_Pad0.74x0.62mm_HandSolder, symbol Device:C
- added C36: 0.1u, Capacitor_SMD:C_0402_1005Metric_Pad0.74x0.62mm_HandSolder, symbol Device:C
- added J10: Conn_01x05_Pin, Connector_PinHeader_2.54mm:PinHeader_1x05_P2.54mm_Vertical, symbol Connector:Conn_01x05_Pin
- added J2: Conn_01x04_Pin, Connector_PinHeader_2.54mm:PinHeader_1x04_P2.54mm_Vertical, symbol Connector:Conn_01x04_Pin
- added J5: Conn_01x02_Pin, Connector_PinHeader_2.00mm:PinHeader_1x02_P2.00mm_Vertical, symbol Connector:Conn_01x02_Pin
- added JP1, JP8: SolderJumper_3_Open, Jumper:SolderJumper-3_P2.0mm_Open_TrianglePad1.0x1.5mm, symbol Jumper:SolderJumper_3_Open
- added JP2, JP3, JP9: SolderJumper_2_Open, Jumper:SolderJumper-2_P1.3mm_Open_TrianglePad1.0x1.5mm, symbol Jumper:SolderJumper_2_Open
- added R51: 10k, Resistor_SMD:R_0402_1005Metric_Pad0.72x0.64mm_HandSolder, symbol Device:R
- added R52: 0, Resistor_SMD:R_0402_1005Metric_Pad0.72x0.64mm_HandSolder, symbol Device:R
- added SW2: SW_Push, Button_Switch_SMD:SW_Push_1P1T-SH_NO_CK_KMR2xxG, symbol Switch:SW_Push
- added U6: ~, display:LED_0.96inch, symbol display:OLED_0.96inch
- C32: value 680u -> 470u; footprint Capacitor_SMD:CP_Elec_10x10.5 -> Capacitor_THT:C_Radial_D6.3mm_H7.0mm_P2.50mm; LSCS Part # (none) -> ROQANG GR1A471M0608
- IC5: footprint ESP32PICOMINI02N8R2 -> ESP32-PICO-MINI-02-N8R2:ESP32PICOMINI02N8R2
Connections:
- net +3.3V: now also C33.2, C34.2, J2.1 (Pin_1), R51.1, U6.3 (VCC)
- net BOOT0: no longer R4.2, U2.45 (PB8)
- net ESP_EN: now also C35.2, R51.2, R52.2
- net GND: now also C33.1, C34.1, C35.1, C36.1, J10.1 (Pin_1), J2.4 (Pin_4), J5.1 (Pin_1), SW2.2, U6.4 (GND)
- net I2C1_SCL: now also U6.2 (SCL); no longer IC5.10 (I35)
- net I2C1_SDA: now also U6.1 (SDA); no longer IC5.9 (I34)
- net TMS: now reaches IC5.18 (IO14)
- net TMS: now also J10.5 (Pin_5), JP9.2 (B)
- net TDI: now reaches IC5.19 (IO12)
- net TDI: now also J10.4 (Pin_4), JP3.2 (B)
- net TCK: now reaches IC5.20 (IO13)
- net TCK: now also J10.3 (Pin_3), JP8.3 (B)
- net TDO: now reaches IC5.21 (IO15)
- net TDO: now also J10.2 (Pin_2), JP1.3 (B)
- net HANDSHAKE_ESP32: now reaches IC5.22 (IO2)
- net HANDSHAKE_ESP32: now also JP2.2 (B)
- net BOOT0_ESP32: now reaches IC5.23 (IO0)
- net BOOT0_ESP32: now also J5.2 (Pin_2)
- net ESP_RX: now reaches IC5.30 (RXD0)
- net ESP_RX: now also J2.2 (Pin_2), JP8.1 (A)
- net ESP_TX: now reaches IC5.31 (TXD0)
- net ESP_TX: now also J2.3 (Pin_3), JP1.1 (A)
- net HANDSHAKE_STM32: now reaches CN10.2 (Pin_2)
- net HANDSHAKE_STM32: now also JP2.1 (A)
- net MISO3/RX3: now reaches CN7.1 (Pin_1)
- net MISO3/RX3: now also JP8.2 (C)
- net SCK3/TX3: now reaches CN7.2 (Pin_2)
- net SCK3/TX3: now also JP1.2 (C)
- net ESP32_CS: now reaches CN7.3 (Pin_3)
- net ESP32_CS: now also JP9.1 (A)
- net MOSI3: now reaches CN7.4 (Pin_4)
- net MOSI3: now also JP3.1 (A)
- new net: C36.2, R52.1, SW2.1
- new net BOOT0_STM32: R4.2, U2.45 (PB8)
- no-connect marks 35 -> 72
Other:
- note added: "BOOT0"
- note added: "CHOOSE COMMUNICATION"
- note added: "ENABLE"
- note added: "ESP32­PICO­MINI­02 DATASHEET"
- note added: "Hardware Reference"
- note added: "JTAG"
- note added: "UART INTERFACE"
- moved on the sheet: IC5

Commit message: added selectable I2C/UART for peripheral (LIDAR), added some annotation for soldermaks
Parts:
- added JP4, JP5: SolderJumper_3_Open, Jumper:SolderJumper-3_P2.0mm_Open_TrianglePad1.0x1.5mm, symbol Jumper:SolderJumper_3_Open
- added JP6, JP7: SolderJumper_2_Open, Jumper:SolderJumper-2_P1.3mm_Open_TrianglePad1.0x1.5mm, symbol Jumper:SolderJumper_2_Open
Connections:
- net I2C1_SCL: now also JP5.3 (B); no longer Q2.3 (D), R12.1
- net I2C1_SCL_5V: now also JP7.1 (A)
- net I2C1_SDA: now also JP4.3 (B); no longer Q1.3 (D), R11.1
- net I2C1_SDA_5V: now also JP6.1 (A)
- net IsenseM1: now also CN7.35 (Pin_35), J14.5 (Pin_5); no longer CN7.27 (Pin_27), J14.1 (Pin_1)
- net IsenseM2: now also CN7.37 (Pin_37), J14.6 (Pin_6); no longer CN7.29 (Pin_29), J14.2 (Pin_2)
- new net I2C1_SCL_SEL: JP5.2 (C), JP7.2 (B), Q2.3 (D), R12.1
- new net I2C1_SDA_SEL: JP4.2 (C), JP6.2 (B), Q1.3 (D), R11.1
- new net UART4_RX: CN7.29 (Pin_29), J14.2 (Pin_2), JP5.1 (A)
- new net UART4_TX: CN7.27 (Pin_27), J14.1 (Pin_1), JP4.1 (A)
Other:
- note added: "SELECT COMM UART or I2C"
- note added: "SELECT VOLTAGE"
- moved on the sheet: C32, LiDAR-V1, Q1, Q2, R11, R12, R22, R23
