File: DAWG_ServoDriver-backups/DAWG_ServoDriver-2024-04-09_195908/DAWG_ServoDriver.kicad_sch (KiCad schematic)
At the start: 156 parts, among them CN10 Conn_02x19_Odd_Even, CN7 Conn_02x19_Odd_Even, IC1 DRV8251ADDAR, IC2 DRV8251ADDAR, IC3 DRV8251ADDAR, IC4 DRV8251ADDAR, IC5 ESP32-PICO-MINI-02-N8R2, J1 Conn_01x05, J10 Screw_Terminal_01x02, J11 Conn_01x10, J12 Conn_01x08, J13 Conn_01x05, J14 Conn_01x06, J15 Conn_01x08, J16 Screw_Terminal_01x02, J17 Conn_01x03, J18 Conn_01x03, J19 Conn_01x03, J2 Screw_Terminal_01x02, J20 Conn_01x03, J21 Conn_01x03, J22 Conn_01x03, J23 Conn_01x03, J24 Conn_01x03, J25 Conn_01x03, J26 Conn_01x03, J27 Conn_01x03, J28 Conn_01x03, J29 Conn_01x03, J3 Conn_01x05, J30 Conn_01x03, J31 Conn_01x03, J32 Conn_01x03, J33 Conn_01x03, J34 Conn_01x03, J35 Conn_01x03, J36 Conn_01x03, J4 Conn_01x04_Pin, J5 Screw_Terminal_01x02, J6 Conn_01x03, J7 Screw_Terminal_01x02, J8 Screw_Terminal_01x02, J9 Conn_01x05, Q1 BSS138, Q10 BSS138, Q11 BSS138, Q12 BSS138, Q13 BSS138, Q14 BSS138, Q15 BSS138, Q16 BSS138, Q17 BSS138, Q18 BSS138, Q19 BSS138, Q2 BSS138, Q20 BSS138, Q3 BSS138, Q4 BSS138, Q5 BSS138, Q6 BSS138, Q7 BSS138, Q8 BSS138, Q9 BSS138, SW1 SW_Push, U1 TPS62177DQC, U2 STM32G431C8Tx, U3 LD1117S12TR_SOT223, U4 ICM-20602, U5 ICM-20602, Y1 Crystal_GND24

Commit message: Finished Routing all except IMU2_INT and GNDs
Parts:
- removed IC5: ESP32-PICO-MINI-02-N8R2, ESP32PICOMINI02N8R2, symbol MCU_Espressif:ESP32-PICO-MINI-02-N8R2
- removed J36: Conn_01x03, Connector_PinHeader_2.54mm:PinHeader_1x03_P2.54mm_Vertical, symbol Connector_Generic:Conn_01x03
- J1, J13, J3, J9: footprint Connector_PinHeader_2.54mm:PinHeader_1x05_P2.54mm_Vertical -> TerminalBlock_MetzConnect:TerminalBlock_MetzConnect_Type011_RT05505HBWC_1x05_P5.00mm_Horizontal
- J10, J16, J2, J5: footprint Connector_PinHeader_2.54mm:PinHeader_1x02_P2.54mm_Vertical -> TerminalBlock_MetzConnect:TerminalBlock_MetzConnect_Type011_RT05502HBWC_1x02_P5.00mm_Horizontal
- J11: footprint Connector_PinHeader_2.54mm:PinHeader_1x10_P2.54mm_Vertical -> Connector_PinHeader_2.54mm:PinHeader_1x10_P2.54mm_Vertical_SMD_Pin1Left
- J12: footprint Connector_PinHeader_2.54mm:PinHeader_1x08_P2.54mm_Vertical -> Connector_PinHeader_2.54mm:PinHeader_1x08_P2.54mm_Vertical_SMD_Pin1Left
- J14: footprint Connector_PinHeader_2.54mm:PinHeader_1x06_P2.54mm_Vertical -> Connector_PinHeader_2.54mm:PinHeader_1x06_P2.54mm_Vertical_SMD_Pin1Left
- J15: footprint Connector_PinHeader_2.54mm:PinHeader_1x08_P2.54mm_Vertical -> Connector_PinHeader_2.54mm:PinHeader_1x08_P2.54mm_Vertical_SMD_Pin1Right
- J18, J21, J24, J27, J30, J33, J6: footprint Connector_PinHeader_2.54mm:PinHeader_1x03_P2.54mm_Vertical -> Connector_PinHeader_2.54mm:PinHeader_1x03_P2.54mm_Vertical_SMD_Pin1Left
- J4: footprint Connector_PinHeader_2.54mm:PinHeader_1x04_P2.54mm_Vertical -> Connector_PinHeader_2.54mm:PinHeader_1x04_P2.54mm_Vertical_SMD_Pin1Left
- LiDAR-V1: footprint Connector_PinHeader_2.54mm:PinHeader_1x05_P2.54mm_Vertical -> Connector_PinHeader_2.54mm:PinHeader_1x05_P2.54mm_Vertical_SMD_Pin1Left
- SW1: footprint Button_Switch_SMD:SW_Push_1P1T-SH_NO_CK_KMR2xxG -> Button_Switch_SMD:SW_DIP_SPSTx02_Slide_6.7x6.64mm_W8.61mm_P2.54mm_LowProfile
- renumbered CN10 to CN1, CN7 to CN2
Connections:
- net GND: no longer CN1.9 (Pin_9), J11.7 (Pin_7)
- net I2C3_SCL: now also U2.30 (PA8)
- net IMU1_INT: now also CN1.12 (Pin_12); no longer CN1.4 (Pin_4)
- net IMU2_INT: now also CN1.16 (Pin_16); no longer CN1.2 (Pin_2)
- net Mtr1_EncoderA: now also CN1.2 (Pin_2); no longer CN1.11 (Pin_11), J11.6 (Pin_6)
- net Mtr1_EncoderB: now also CN1.4 (Pin_4); no longer CN1.17 (Pin_17), J11.3 (Pin_3)
- net Mtr1_EncoderZ: now also CN1.14 (Pin_14); no longer CN1.16 (Pin_16)
- net Mtr2_EncoderA: now also CN1.22 (Pin_22); no longer CN1.29 (Pin_29), J15.5 (Pin_5)
- net Mtr2_EncoderB: now also CN1.26 (Pin_26); no longer CN1.31 (Pin_31), J15.4 (Pin_4)
- net Mtr3_EncoderA: now also CN1.33 (Pin_33), J15.3 (Pin_3); no longer CN2.23 (Pin_23)
- net Mtr3_EncoderB: now also CN1.31 (Pin_31), J15.4 (Pin_4); no longer CN2.21 (Pin_21)
- net Mtr3_EncoderZ: now also CN1.27 (Pin_27), J15.6 (Pin_6); no longer CN2.17 (Pin_17)
- net Mtr4_EncoderA: now also CN2.17 (Pin_17); no longer CN1.26 (Pin_26)
- net Mtr4_EncoderB: now also CN2.21 (Pin_21); no longer CN1.24 (Pin_24)
- net Mtr4_EncoderZ: now also CN2.23 (Pin_23); no longer CN1.22 (Pin_22)
- net PWM15/1: now also Q18.2 (S), R48.1; no longer Q12.2 (S), R42.1
- net PWM15/2: now also Q19.2 (S), R49.1, U2.11 (PA3); no longer Q11.2 (S), R32.1, U2.29 (PB15)
- net PWM16/1: now also Q20.2 (S), R50.1; no longer Q5.2 (S), R26.1
- net PWM1/1: now also Q3.2 (S), R24.1, U2.15 (PA7); no longer Q10.2 (S), R31.1, U2.30 (PA8)
- net PWM1/2: now also Q4.2 (S), R25.1; no longer Q9.2 (S), R30.1
- net PWM1/3: now also Q5.2 (S), R26.1; no longer Q8.2 (S), R29.1
- net PWM1/4: now also Q6.2 (S), R27.1; no longer Q7.2 (S), R28.1
- net PWM2/1: now also CN2.28 (Pin_28), J14.1 (Pin_1), Q7.2 (S), R28.1; no longer Q17.2 (S), R47.1
- net PWM2/1_M1: now also CN1.11 (Pin_11), J11.6 (Pin_6); no longer CN1.13 (Pin_13), J11.5 (Pin_5)
- net PWM2/2: now also CN2.30 (Pin_30), J14.2 (Pin_2), Q8.2 (S), R29.1; no longer Q20.2 (S), R50.1
- net PWM2/3: now also Q9.2 (S), R30.1; no longer Q19.2 (S), R49.1
- net PWM2/4: now also Q10.2 (S), R31.1; no longer Q13.2 (S), R43.1
- net PWM3/1: now also Q11.2 (S), R32.1; no longer Q16.2 (S), R46.1
- net PWM3/1_M1: now also CN1.13 (Pin_13), J11.5 (Pin_5); no longer CN1.15 (Pin_15), J11.4 (Pin_4)
- net PWM3/2: now also Q12.2 (S), R42.1; no longer Q18.2 (S), R48.1
- net PWM3/2_M2: now also CN1.19 (Pin_19), J11.2 (Pin_2); no longer CN1.27 (Pin_27), J15.6 (Pin_6)
- net PWM3/2_M4: now also CN1.29 (Pin_29), J15.5 (Pin_5); no longer CN1.33 (Pin_33), J15.3 (Pin_3)
- net PWM3/3: now also Q13.2 (S), R43.1; no longer Q15.2 (S), R45.1
- net PWM4/1: now also Q15.2 (S), R45.1; no longer Q4.2 (S), R25.1
- net PWM4/1_M2: now also CN1.17 (Pin_17), J11.3 (Pin_3); no longer CN1.19 (Pin_19), J11.2 (Pin_2)
- net PWM4/2: now also Q16.2 (S), R46.1; no longer Q6.2 (S), R27.1
- net PWM4/4: now also Q17.2 (S), R47.1; no longer Q3.2 (S), R24.1
- net ADC1/14: now reaches CN1.34 (Pin_34)
- net ADC1/14: now also IC1.1 (IPROPI), R1.2
- net ADC1/15: now reaches CN1.6 (Pin_6)
- net ADC1/15: now also IC2.1 (IPROPI), R3.2
- removed net IsenseM1: CN2.28 (Pin_28), IC1.1 (IPROPI), J14.1 (Pin_1), R1.2
- removed net IsenseM2: CN2.30 (Pin_30), IC2.1 (IPROPI), J14.2 (Pin_2), R3.2
- net IsenseM3 renamed ADC1/9
- net ADC1/9: now also CN1.24 (Pin_24); no longer CN2.34 (Pin_34), J14.4 (Pin_4)
- net IsenseM4: no longer names the net of CN2.32 (Pin_32), J14.3 (Pin_3)
- net IsenseM4: no longer IC4.1 (IPROPI), R10.2
- new net: CN1.9 (Pin_9), J11.7 (Pin_7)
- new net ADC1/7: CN1.15 (Pin_15), IC4.1 (IPROPI), J11.4 (Pin_4), R10.2
- new net PWM1/2N: CN2.34 (Pin_34), J14.4 (Pin_4)
- no-connect marks 43 -> 44
Other:
- note removed: "DONE"
- note removed: "ESP32-PICO-MINI-02"
- moved on the sheet: C18, C19, CN2, D1, D2, J12, J14, J7, J8, R5, R6
