File: DAWG_ServoDriver-backups/DAWG_ServoDriver-2024-04-10_225434/DAWG_ServoDriver.kicad_sch (KiCad schematic)
At the start: 154 parts, among them CN10 Conn_02x19_Odd_Even, CN7 Conn_02x19_Odd_Even, IC1 DRV8251ADDAR, IC2 DRV8251ADDAR, IC3 DRV8251ADDAR, IC4 DRV8251ADDAR, IC5 ESP32-PICO-MINI-02-N8R2, J1 Screw_Terminal_01x06, J11 Conn_01x10, J12 Conn_01x08, J13 Screw_Terminal_01x06, J14 Conn_01x06, J15 Conn_01x08, J17 Conn_01x03, J18 Conn_01x03, J19 Conn_01x03, J2 Conn_01x04, J20 Conn_01x03, J21 Conn_01x03, J22 Conn_01x03, J23 Conn_01x03, J24 Conn_01x03, J25 Conn_01x03, J26 Conn_01x03, J27 Conn_01x03, J28 Conn_01x03, J29 Conn_01x03, J3 Screw_Terminal_01x06, J30 Conn_01x03, J31 Conn_01x03, J32 Conn_01x03, J33 Conn_01x03, J34 Conn_01x03, J35 Conn_01x03, J36 Conn_01x03, J4 Conn_01x04_Pin, J5 Conn_01x04, J6 Conn_01x03, J7 Screw_Terminal_01x02, J8 Screw_Terminal_01x02, J9 Screw_Terminal_01x06, Q1 BSS138, Q10 BSS138, Q11 BSS138, Q12 BSS138, Q13 BSS138, Q14 BSS138, Q15 BSS138, Q16 BSS138, Q17 BSS138, Q18 BSS138, Q19 BSS138, Q2 BSS138, Q20 BSS138, Q3 BSS138, Q4 BSS138, Q5 BSS138, Q6 BSS138, Q7 BSS138, Q8 BSS138, Q9 BSS138, SW1 SW_Push, U1 TPS62177DQC, U2 STM32G431C8Tx, U3 LD1117S12TR_SOT223, U4 ICM-20602, U5 ICM-20602, Y1 Crystal_GND24

Commit message: Key components placed, Onion board begins.
Parts:
- removed J2, J5: Conn_01x04, symbol Connector_Generic:Conn_01x04
Connections:
- net I2C1_SDA_5V is gone; now on net I2C3_SDA: LiDAR-V1.3 (SDA), Q1.2 (S), R22.1
- net +3.3V: no longer IC5.3 (3V3)
- net GND: no longer IC5.1 (GND_1), IC5.11 (GND_3), IC5.14 (GND_4), IC5.2 (GND_2), U1.11 (PAD)
- net I2C1_SCL: no longer IC5.10 (I35)
- net I2C1_SDA: no longer IC5.9 (I34)
- net Mtr3_EncoderA: now also CN10.12 (Pin_12), J11.6 (Pin_6); no longer CN10.32 (Pin_32), J15.4 (Pin_4)
- net Mtr3_EncoderB: now also CN10.18 (Pin_18), J11.3 (Pin_3); no longer CN10.30 (Pin_30), J15.5 (Pin_5)
- net Mtr4_EncoderA: now also CN10.30 (Pin_30), J15.5 (Pin_5); no longer CN10.12 (Pin_12), J11.6 (Pin_6)
- net Mtr4_EncoderB: now also CN10.32 (Pin_32), J15.4 (Pin_4); no longer CN10.18 (Pin_18), J11.3 (Pin_3)
- net PWM1/1_M3: now also CN10.14 (Pin_14), J11.5 (Pin_5); no longer CN10.20 (Pin_20), J11.2 (Pin_2)
- net PWM1/2_M3: now also CN10.16 (Pin_16), J11.4 (Pin_4); no longer CN10.28 (Pin_28), J15.6 (Pin_6)
- net PWM2/3_M4: now also CN10.28 (Pin_28), J15.6 (Pin_6); no longer CN10.14 (Pin_14), J11.5 (Pin_5)
- net PWM3/2_M4: now also CN10.20 (Pin_20), J11.2 (Pin_2); no longer CN10.16 (Pin_16), J11.4 (Pin_4)
- net I2C3_SDA: now reaches U2.42 (PB5)
- net ESP_EN: no longer names the net of IC5.7 (I39)
- net I2C1_SCL_5V renamed I2C3_SCL
- no-connect marks 35 -> 38
Other:
- moved on the sheet: D1, D2, J4, Q1, Q2, R11, R12, R22, R23, R5, R6
